Commit message: Add xacro parameters to tune controller period in simulation.

File: lwr_description/model/kuka_lwr.gazebo.xacro (robot description, xacro)
@@ -1,8 +1,11 @@
 <?xml version="1.0"?>
 <robot xmlns:xacro="http://www.ros.org/wiki/xacro">
-	<xacro:macro name="kuka_lwr_gazebo" params="name">
+	<xacro:macro name="kuka_lwr_gazebo" params="name control_period:=0">
 		<gazebo>
 			<plugin name="${name}_lwr_hw_sim" filename="liblwr_hw_gazebo_plugin.so">
 				<robotNamespace>${name}</robotNamespace>
+				<xacro:if value="${control_period > 0}">
+					<controlPeriod>${control_period}</controlPeriod>
+				</xacro:if>
 			</plugin>
 		</gazebo>

File: lwr_description/model/kuka_lwr.urdf.xacro (robot description, xacro)
@@ -19,5 +19,5 @@
 	<xacro:property name="rate_stiffness" value="20000"/> <!-- reflex to stiffness -->
 	<!-- URDF model /-->
-	<xacro:macro name="kuka_lwr" params="parent name *origin">
+	<xacro:macro name="kuka_lwr" params="parent name gazebo_control_period:=0 *origin">
 		<!-- First (shoulder) element of the arm. Fixed to its parent. -->
 		<joint name="${parent}_${name}_base_joint" type="fixed">
@@ -366,5 +366,5 @@
 			</collision>
 		</link>
-		<xacro:kuka_lwr_gazebo name="${name}"/>
+		<xacro:kuka_lwr_gazebo name="${name}" control_period="${gazebo_control_period}"/>
 		<xacro:kuka_lwr_transmission name="${name}"/>
 	</xacro:macro>
